File: pcb-rf-only/radio103.sch (EAGLE design)
At the start: 71 parts, among them IC1 LM833D, IC2 7805TV, IC3 74ACT00D, IC5 LM386M-1, IC6 LM1117MPX-3.3, J1 PJ-324MH, J2 PJ-324MH, J3 PJ-324MH, U1 FST3253

Commit message: MCP encoder + mic amp
Parts:
- added C28, C31: 100n, rcl:C-EUC0805K
- added C29, C30, C32: (no value), rcl:CPOL-EUE2,5-6E
- added IC7: 4066D, 40xx:4066D
- added IC8: LM833D, linear:LM833D
- added JP4: (no value), pinhead:PINHD-1X2
- added R34, R35, R36, R37, R38, R39, R40: (no value), rcl:R-EU_R0805
Connections:
- new net MIC: IC7C.A
- new net N$48: C30.+, IC8A.+IN, R35.2, R36.1
- new net N$49: C31.1, IC8A.-IN, R34.2, R37.2
- new net N$50: C31.2, IC8A.OUT, R34.1, R39.2
- new net N$51: C29.-, R37.1
- new net N$52: C29.+, JP4.2, R38.2
- new net N$53: C32.-, R39.1
- new net N$54: C32.+, R40.1
- new net RXEN: IC7A.C, IC7B.C
- new net RX_I: IC7A.A
- new net RX_Q: IC7B.A
- new net TXEN: IC7C.C, IC7D.C
- net ADC_RX_I: now also IC7A.B, IC7C.B
- net ADC_RX_Q: now also IC7B.B, IC7D.B
- net GND: now also C28.1, C30.-, IC7D.A, IC8P.V-, JP4.1, R36.2, R40.2
- net VOPAMP: now also C28.2, IC8P.V+, R35.1, R38.1
Other:
- note added: "SWR FWD?"

Commit message: fonts + font generator + UI layout
Changed lines of the file:
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@@
 <sheets>
-<sheet>
-<description>cpu</description>
-<plain>
-</plain>
-<instances>
-</instances>
-<busses>
-</busses>
-<nets>
-</nets>
-</sheet>
 <sheet>
 <description>mixer</description>
