File: pcb/radio103.brd (EAGLE design)
At the start: 99 x 100 mm, 85 parts, among them IC1 LM833D, IC2 7805TV, IC3 74ACT00D, IC4 MCP23S17SO, IC5 LM386M-1, IC6 LM1117MPX-3.3, IC7 4066D, J1 PJ-324MH, J2 PJ-324MH, J3 PJ-324MH, SW1 EC12E_SW, SW2 EC12E_SW, T1 BC847, U1 FST3253

Commit message: MCP encoder + mic amp
Parts:
- added C28, C31: 100n, rcl:C0805K
- added C29, C30, C32: (no value), rcl:E2,5-6E
- added CON1: XT30PW-M, amass:XT30PW-M
- added D4: BAT54S, diode:SOT23
- added H3, H4, H5: MOUNT-HOLE3.0, holes:3,0
- added IC8: LM833D, linear:SO08
- added JP4: (no value), pinhead:1X02
- added R25, R26, R27, R28, R29, R30, R31, R32, R33, R34, R35, R36, R37, R38, R39, R40: (no value), rcl:R0805
- added S1, S2, S3, S4: (no value), switch-omron:B3F-10XX
- moved R14 151.8 mm to (155.6, 87.6), flipped to the bottom
- moved R15 146.7 mm to (153.0, 95.2), flipped to the bottom
- moved D1 144.2 mm to (151.8, 86.4), flipped to the bottom
- moved D2 144.2 mm to (151.8, 66.0), flipped to the bottom
- moved D3 144.2 mm to (151.8, 91.4), flipped to the bottom
- moved H1 137.5 mm to (94.5, 4.57)
- moved C11 136.5 mm to (148.0, 74.9), flipped to the bottom
- moved C12 136.5 mm to (148.0, 64.8), flipped to the bottom
- moved R10 136.5 mm to (148.0, 92.7), flipped to the bottom
- moved R11 136.5 mm to (148.0, 72.4), flipped to the bottom
- moved R12 136.5 mm to (148.0, 69.8), flipped to the bottom
- moved R13 136.5 mm to (148.0, 67.3), flipped to the bottom
- moved R7 136.5 mm to (148.0, 87.6), flipped to the bottom
- moved R8 136.5 mm to (148.0, 85.1), flipped to the bottom
- moved R9 136.5 mm to (148.0, 90.2), flipped to the bottom
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Connections:
- removed net ADC_MIC: U$1.A2
- removed net GND1: U$1.GND
- new net +: CON1.+
- new net -: CON1.-
- new net N$42: R26.1, R27.2, S2.1, S2.2
- new net N$43: R31.1, R32.2, R33.1
- new net N$44: R27.1, R28.2, S3.1, S3.2
- new net N$45: R28.1, R29.2, S4.1, S4.2
- new net N$46: R29.1, R30.2, SW1.D
- new net N$47: R30.1, SW2.D
- new net N$48: C30.+, IC8.3, R35.2, R36.1
- new net N$49: C31.1, IC8.2, R34.2, R37.2
- new net N$50: C31.2, IC8.1, R34.1, R39.2
- new net N$51: C29.-, R37.1
- new net N$52: C29.+, JP4.2, R38.2
- new net N$53: C32.-, R39.1
- new net N$54: C32.+, R40.1
- new net VBAT: R31.2
- net 3V3: now also D4.2, R25.2, U$1.3V3
- net ADC_BTN: now also R25.1, R26.2, S1.1, S1.2
- net ADC_VIN: now also R33.2
- net GND: now also C28.1, C30.-, D4.1, IC8.4, JP4.1, R32.1, R36.2, R40.2, S1.3, S1.4, S2.3, S2.4, S3.3, S3.4, S4.3, S4.4, SW1.E, SW2.E, U$1.GND, U$1.GND1
- net RESET: now also U$1.RESET
- net RXEN: now also R23.1, T1.3; no longer R24.2
- net TXEN: now also R24.2; no longer R23.1, T1.3
- net VOPAMP: now also C28.2, IC8.8, R35.1, R38.1

Commit message: fonts + font generator + UI layout
Parts:
- added D5, D6, D7, D8: BAT54S, diode:SOT23
- added IC10: 78L05Z, linear:TO92
- added IC9: 78L08Z, linear:TO92
- added R41, R42, R43, R44: (no value), rcl:R0805
- moved C28 92.1 mm to (41.3, -160.7), flipped to the bottom
- moved C31 92.1 mm to (41.3, -207.0), flipped to the bottom
- moved R34 90.8 mm to (40.6, -166.4), flipped to the bottom
- moved R35 90.8 mm to (40.6, -170.8), flipped to the bottom
- moved R36 90.8 mm to (40.6, -175.3), flipped to the bottom
- moved R37 90.8 mm to (40.6, -179.7), flipped to the bottom
- moved R38 90.8 mm to (40.6, -190.5), flipped to the bottom
- moved R39 90.8 mm to (40.6, -212.7), flipped to the bottom
- moved R40 90.8 mm to (40.6, -223.5), flipped to the bottom
- moved C29 89.5 mm to (40.0, -184.2), flipped to the bottom
- moved C30 89.5 mm to (40.0, -201.3), flipped to the bottom
- moved C32 89.5 mm to (40.0, -217.2), flipped to the bottom
- moved JP4 89.5 mm to (40.0, -195.6), flipped to the bottom
- moved IC8 87.0 mm to (38.7, -153.7), flipped to the bottom
- moved D4 73.0 mm to (31.8, -150.5), flipped to the bottom
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Connections:
- new net N$55: D5.3, IC4.25, R43.1
- new net N$56: R43.2
- new net N$57: D6.3, IC4.26, R41.1
- new net N$58: R41.2
- new net N$59: D7.3, IC4.27, R42.1
- new net N$60: R42.2
- new net N$61: D8.3, IC4.28, R44.1
- new net N$62: R44.2
- net 3V3: now also D5.2, D6.2, D7.2, D8.2
- net GND: now also D5.1, D6.1, D7.1, D8.1
- net N$43: now also D4.3

Commit message: gfx improved
Parts:
- added C33, C34, C35, C36, C37, C38: 100n, rcl:C0805K
- added IC11: LM833D, linear:SO08
- added R45, R46, R47, R48, R49, R50: (no value), rcl:R0805
Connections:
- new net N$63: C33.2, IC11.3, R45.2
- new net N$64: C35.1, R45.1, R46.2
- new net N$65: C35.2, IC11.1, IC11.2, R50.1
- new net N$66: C38.1, R48.1, R49.2
- new net N$67: C34.2, R46.1, R47.2
- new net N$68: R47.1
- new net N$69: C37.2, R49.1, R50.2
- new net N$71: C36.2, IC11.5, R48.2
- new net N$73: C38.2, IC11.6, IC11.7
- new net V+: IC11.8
- new net V-: IC11.4
- net GND: now also C33.1, C34.1, C36.1, C37.1

Commit message: menu system + splash RLE
Parts:
- removed IC4: MCP23S17SO, microchip:SO28W
- added IC12: 74HC595D, 74xx-eu:SO16
- moved U$4 38.1 mm to (35.6, 54.0), turned to 180 degrees
- moved S4 4.45 mm to (57.1, 5.71)
- moved S3 3.81 mm to (43.8, 5.71)
- moved S2 2.54 mm to (29.8, 5.71)
Connections:
- net ONBOARD_LED renamed LED_BUILTIN
- new net ADC_RESERVED: U$1.A6
- net 3V3: now also IC12.16; no longer IC4.9
- net ADC_BTN: now also U$1.A2; no longer U$1.A3
- net ADC_SWR_F: now also U$1.A3; no longer U$1.A4
- net ADC_SWR_R: now also U$1.A4; no longer U$1.A5
- net ADC_VIN: now also U$1.A5; no longer U$1.A6
- net EXP_CS: now also IC12.12, U$1.A9; no longer IC4.11
- net GND: now also IC12.13, IC12.8; no longer IC4.10, IC4.15, IC4.16, IC4.17
- net LCD_CS: now also U$1.A12
- net LCD_DC: now also U$1.A15
- net N$16: no longer IC4.21
- net N$38: no longer IC4.22
- net N$40: no longer IC4.23
- net N$41: no longer IC4.24
- net N$55: now also IC12.15; no longer IC4.25
- net N$57: now also IC12.1; no longer IC4.26
- net N$59: now also IC12.2; no longer IC4.27
- net N$61: now also IC12.3; no longer IC4.28
- net RESET: no longer IC4.18
- net SCL: now also U$1.B10; no longer U$1.B8
- net SDA: now also U$1.B11; no longer U$1.B9
- net SPI_MISO: no longer IC4.14
- net SPI_MOSI: now also IC12.14; no longer IC4.13
- net SPI_SCK: now also IC12.11; no longer IC4.12

Commit message: test
Parts:
- moved C33 144.9 mm to (62.9, -178.4), flipped to the bottom
- moved C34 144.9 mm to (62.9, -183.5), flipped to the bottom
- moved C35 144.9 mm to (62.9, -188.6), flipped to the bottom
- moved C36 144.9 mm to (62.9, -193.7), flipped to the bottom
- moved C38 144.9 mm to (62.9, -212.1), flipped to the bottom
- moved R45 144.1 mm to (62.2, -165.7), flipped to the bottom
- moved R46 144.1 mm to (62.2, -170.2), flipped to the bottom
- moved R47 144.1 mm to (62.2, -174.6), flipped to the bottom
- moved R48 144.1 mm to (62.2, -199.4), flipped to the bottom
- moved R49 144.1 mm to (62.2, -203.8), flipped to the bottom
- moved R50 144.1 mm to (62.2, -208.3), flipped to the bottom
- moved IC11 141.9 mm to (60.3, -158.1), flipped to the bottom
- moved C37 139.7 mm to (58.4, -193.7), flipped to the bottom
- moved IC12 138.3 mm to (57.1, -219.7), flipped to the bottom
- moved R42 134.2 mm to (53.3, -149.2), flipped to the bottom
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Connections:
- net N$55: no longer IC12.15
- net N$57: no longer IC12.1
- net N$59: no longer IC12.2
- net N$61: no longer IC12.3
